File: eagle/clock.sch (EAGLE design)
At the start: 55 parts, among them CN1 ARDUINO_SHIELDNO_SILK, IC1 TPS55330TRE, IC2 TCS3472FN, Q1 BC817-40SMD, Q2 SUD50P04-13L

Commit message: started work on the layout. PSU is layed out too
Connections:
- net N$1 renamed FREQ
- net N$2 renamed SS
- net N$20 renamed LED12
- net N$22 renamed LED15
- net N$3 renamed SW
- net N$4 renamed FB
- net N$6 renamed COMP

Commit message: came up with a better location for the buttons
Connections:
- removed net N$26: CN1.A0, LEFT.1
- removed net N$27: CN1.A1, DOWN.1
- removed net N$28: CN1.A2, UP.1
- removed net N$29: CN1.A3, RIGHT.1
- new net N$1: CN1.A3, LEFT.1
- new net N$2: CN1.A2, DOWN.1
- new net N$3: CN1.A1, UP.1
- new net N$4: CN1.A0, RIGHT.1
Other:
- moved on the sheet: DOWN, LEFT, RIGHT, UP
Changed lines of the file:
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@@
 <attribute name="VALUE" x="209.55" y="-43.18" size="1.778" layer="96"/>
 </instance>
-<instance part="LEFT" gate="G$1" x="198.12" y="-2.54"/>
-<instance part="DOWN" gate="G$1" x="198.12" y="-5.08"/>
-<instance part="UP" gate="G$1" x="198.12" y="-7.62"/>
-<instance part="RIGHT" gate="G$1" x="198.12" y="-10.16"/>
+<instance part="LEFT" gate="G$1" x="200.66" y="-10.16"/>
+<instance part="DOWN" gate="G$1" x="200.66" y="-7.62"/>
+<instance part="UP" gate="G$1" x="200.66" y="-5.08"/>
+<instance part="RIGHT" gate="G$1" x="200.66" y="-2.54"/>
 <instance part="LED0" gate="G$1" x="63.5" y="-66.04" smashed="yes">
 <attribute name="NAME" x="53.34" y="-73.66" size="1.778" layer="95"/>
@@
 </segment>
 </net>
-<net name="N$26" class="0">
-<segment>
-<pinref part="CN1" gate="G$1" pin="A0"/>
-<wire x1="205.74" y1="-2.54" x2="203.2" y2="-2.54" width="0.1524" layer="91"/>
-<pinref part="LEFT" gate="G$1" pin="1"/>
-</segment>
-</net>
-<net name="N$27" class="0">
-<segment>
-<pinref part="CN1" gate="G$1" pin="A1"/>
-<wire x1="205.74" y1="-5.08" x2="203.2" y2="-5.08" width="0.1524" layer="91"/>
-<pinref part="DOWN" gate="G$1" pin="1"/>
-</segment>
-</net>
-<net name="N$28" class="0">
-<segment>
-<pinref part="CN1" gate="G$1" pin="A2"/>
-<wire x1="205.74" y1="-7.62" x2="203.2" y2="-7.62" width="0.1524" layer="91"/>
-<pinref part="UP" gate="G$1" pin="1"/>
-</segment>
-</net>
-<net name="N$29" class="0">
-<segment>
-<pinref part="CN1" gate="G$1" pin="A3"/>
-<wire x1="205.74" y1="-10.16" x2="203.2" y2="-10.16" width="0.1524" layer="91"/>
-<pinref part="RIGHT" gate="G$1" pin="1"/>
-</segment>
-</net>
 <net name="N$5" class="0">
 <segment>
@@
 </segment>
 </net>
+<net name="N$1" class="0">
+<segment>
+<pinref part="CN1" gate="G$1" pin="A3"/>
+<pinref part="LEFT" gate="G$1" pin="1"/>
+</segment>
+</net>
+<net name="N$2" class="0">
+<segment>
+<pinref part="CN1" gate="G$1" pin="A2"/>
+<pinref part="DOWN" gate="G$1" pin="1"/>
+</segment>
+</net>
+<net name="N$3" class="0">
+<segment>
+<pinref part="CN1" gate="G$1" pin="A1"/>
+<pinref part="UP" gate="G$1" pin="1"/>
+</segment>
+</net>
+<net name="N$4" class="0">
+<segment>
+<pinref part="CN1" gate="G$1" pin="A0"/>
+<pinref part="RIGHT" gate="G$1" pin="1"/>
+</segment>
+</net>

Commit message: Almost finished layout
Parts:
- added C19: 10uF, rcl:C-EUC1206K
- added R9: 1k, rcl:R-US_R0603
Connections:
- new net N$6: CN1.TX, R9.1
- net GND: now also C19.2
- net LIGHT-INT: now also R9.2; no longer CN1.D7
- net PWR-EN: now also CN1.A5; no longer CN1.*D9
- net SMPSU-OUTPUT: now also C19.1
Other:
- moved on the sheet: C10, DOWN, IC2, LEFT, Q1, Q2, R5, R6, R7, R8, RIGHT, UP
